Commit message: trying to plan

File: xacro/gummi_base.srdf.xacro (robot description, xacro)
@@ -9,5 +9,5 @@
   <joint name="left_upperarm_roll" />
   <joint name="left_elbow" />
-  <joint name="fastswitch" />
+  <joint name="left_fastswitch" />
 </xacro:macro>
 <xacro:macro name="group_state_left_arm_base">
