Commit message: it moves

File: urdf/gummi_description.urdf (robot description, URDF)
Before this commit: robot gummi, 21 links, 20 joints
Links:
- added link base_link
Joints:
- added joint leftbase_displacement: type fixed, parent base_link, child left_base_link, origin xyz=-0.2 0 0 rpy=-3.14 0 0, axis 0 0 0

File: xacro/gummi_left.urdf.xacro (robot description, xacro)
@@ -4,10 +4,3 @@
 <xacro:include filename="$(env GUMMI_LEFTBASEPATH)/xacro/gummi_description_base.urdf.xacro" />
 <xacro:include filename="$(env GUMMI_LEFTEEPATH)/xacro/gummi_description_ee.urdf.xacro" />
-<link name="base_link"/>
-<joint name="leftbase_displacement" type="fixed">
-  <origin rpy="-3.14 0 0" xyz="-0.2 0 0"/>
-  <parent link="base_link"/>
-  <child link="left_base_link"/>
-  <axis xyz="0 0 0"/>
-</joint>
 </robot>

Commit message: changes for namespaceing /left

File: urdf/gummi_description.urdf (robot description, URDF)
Before this commit: robot gummi, 22 links, 21 joints
Links:
- removed link dummyleft_gripper
- removed link left_base_link
- removed link left_i1
- removed link left_i2
- removed link left_i3
- removed link left_i4
- removed link left_i5
- removed link left_lowerarm
- removed link left_lowerarm_preroll_d
- removed link left_lowerarm_preroll_u
- removed link left_shoulder
- removed link left_shoulder_pitch_back_pulley
- removed link left_shoulder_pitch_front_pulley
- removed link left_shoulder_preroll
- removed link left_shoulder_roll_bottom_pulley
- removed link left_shoulder_roll_top_pulley
- removed link left_upperarm
- removed link left_upperarm_biceps_pulley
- removed link left_upperarm_preroll
- removed link left_upperarm_triceps_pulley
- removed link left_wrist
- added link dummyleft/gripper
- added link left/base_link, mass 0.335467320988356; collision mesh filename=package://gummi_leftbase_template/meshes/base_link.STL; visual mesh filename=package://gummi_leftbase_template/meshes/base_link.STL
- added link left/i1, mass 0.00632408233084942; collision mesh filename=package://gummi_leftee_handshake/meshes/i1.STL; visual mesh filename=package://gummi_leftee_handshake/meshes/i1.STL
- added link left/i2, mass 0.00478605585780196; collision mesh filename=package://gummi_leftee_handshake/meshes/i2.STL; visual mesh filename=package://gummi_leftee_handshake/meshes/i2.STL
- added link left/i3, mass 0.00575461720344836; collision mesh filename=package://gummi_leftee_handshake/meshes/i3.STL; visual mesh filename=package://gummi_leftee_handshake/meshes/i3.STL
- added link left/i4, mass 0.00478456052942582; collision mesh filename=package://gummi_leftee_handshake/meshes/i4.STL; visual mesh filename=package://gummi_leftee_handshake/meshes/i4.STL
- added link left/i5, mass 0.00396686667442233; collision mesh filename=package://gummi_leftee_handshake/meshes/i5.STL; visual mesh filename=package://gummi_leftee_handshake/meshes/i5.STL
- added link left/lowerarm, mass 0.214658222402075; collision mesh filename=package://gummi_leftee_handshake/meshes/lowerarm.STL; visual mesh filename=package://gummi_leftee_handshake/meshes/lowerarm.STL
- added link left/lowerarm_preroll_d, mass 0.0573922743530686; collision mesh filename=package://gummi_leftee_handshake/meshes/lowerarm_preroll_d.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; visual mesh filename=package://gummi_leftee_handshake/meshes/lowerarm_preroll_d.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
- added link left/lowerarm_preroll_u, mass 0.034447; collision mesh filename=package://gummi_leftbase_template/meshes/lowerarm_preroll_u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; visual mesh filename=package://gummi_leftbase_template/meshes/lowerarm_preroll_u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
- added link left/shoulder, mass 0.32611; collision mesh filename=package://gummi_leftbase_template/meshes/shoulder.STL; visual mesh filename=package://gummi_leftbase_template/meshes/shoulder.STL
- added link left/shoulder_pitch_back_pulley, mass 0.027251; collision mesh filename=package://gummi_leftbase_template/meshes/shoulder_pitch_bac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; visual mesh filename=package://gummi_leftbase_template/meshes/shoulder_pitch_bac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
- added link left/shoulder_pitch_front_pulley, mass 0.027251; collision mesh filename=package://gummi_leftbase_template/meshes/shoulder_pitch_fro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; visual mesh filename=package://gummi_leftbase_template/meshes/shoulder_pitch_fro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
- added link left/shoulder_preroll, mass 0.77225; collision mesh filename=package://gummi_leftbase_template/meshes/shoulder_preroll.S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; visual mesh filename=package://gummi_leftbase_template/meshes/shoulder_preroll.S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
- added link left/shoulder_roll_bottom_pulley, mass 0.01522; collision mesh filename=package://gummi_leftbase_template/meshes/shoulder_roll_bott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; visual mesh filename=package://gummi_leftbase_template/meshes/shoulder_roll_bott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
- added link left/shoulder_roll_top_pulley, mass 0.01522; collision mesh filename=package://gummi_leftbase_template/meshes/shoulder_roll_top_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; visual mesh filename=package://gummi_leftbase_template/meshes/shoulder_roll_top_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
- added link left/upperarm, mass 0.26501; collision mesh filename=package://gummi_leftbase_template/meshes/upperarm.STL; visual mesh filename=package://gummi_leftbase_template/meshes/upperarm.STL
- added link left/upperarm_biceps_pulley, mass 0.01522; collision mesh filename=package://gummi_leftbase_template/meshes/upperarm_biceps_pu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; visual mesh filename=package://gummi_leftbase_template/meshes/upperarm_biceps_pu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
- added link left/upperarm_preroll, mass 0.11889; collision mesh filename=package://gummi_leftbase_template/meshes/upperarm_preroll.S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; visual mesh filename=package://gummi_leftbase_template/meshes/upperarm_preroll.S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
- added link left/upperarm_triceps_pulley, mass 0.01522; collision mesh filename=package://gummi_leftbase_template/meshes/upperarm_triceps_p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; visual mesh filename=package://gummi_leftbase_template/meshes/upperarm_triceps_p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
- added link left/wrist, mass 0.0644774651698934; collision mesh filename=package://gummi_leftee_handshake/meshes/wrist.STL; visual mesh filename=package://gummi_leftee_handshake/meshes/wrist.STL
Joints:
- removed joint left_elbow
- removed joint left_fastswitch
- removed joint left_forearm_roll
- removed joint left_gripper
- removed joint left_i1f
- removed joint left_i2f
- removed joint left_i3f
- removed joint left_i4f
- removed joint left_i5f
- removed joint left_shoulder_pitch
- removed joint left_shoulder_pitch_back_pulley_joint
- removed joint left_shoulder_pitch_pulley_front_joint
- removed joint left_shoulder_roll
- removed joint left_shoulder_roll_bottom_pulley
- removed joint left_shoulder_roll_top_pulley_joint
- removed joint left_shoulder_yaw
- removed joint left_upperarm_biceps_pulley_joint
- removed joint left_upperarm_roll
- removed joint left_upperarm_triceps_pulley_joint
- removed joint left_wrist_pitch
- added joint left/elbow: type revolute, parent left/upperarm, child left/lowerarm_preroll_u, origin xyz=-0.006 0.0184 -0.23533 rpy=0 0 0, axis 0 -1 0, limit lower=-0.75 upper=0.35 effort=0 velocity=0
- added joint left/fastswitch: type fixed, parent left/lowerarm_preroll_u, child left/lowerarm_preroll_d, origin xyz=0.056236 -0.019 -0.006 rpy=0 0 0, axis 0 0 0
- added joint left/forearm_roll: type continuous, parent left/lowerarm_preroll_d, child left/lowerarm, origin xyz=0.043506 -0.00023376 -0.019876 rpy=0 0 0, axis -1 0 0, limit effort=0 velocity=1
- added joint left/gripper: type revolute, parent left/wrist, child dummyleft/gripper, origin xyz=0 0 0 rpy=0 0 0, axis 0 1 0, limit lower=0 upper=2 effort=0 velocity=0
- added joint left/i1f: type revolute, parent left/wrist, child left/i1, origin xyz=0.059922 -0.031986 0.0029515 rpy=-0.79367 0.12795 -0.91441, axis 0 -1 0, limit lower=0 upper=0.8 effort=0 velocity=0, mimic joint=left/gripper
- added joint left/i2f: type revolute, parent left/wrist, child left/i2, origin xyz=0.12886 -0.0060786 -0.0024749 rpy=-6.9389E-16 -8.4436E-17 -0.12109, axis 0 -1 0, limit lower=0 upper=0.8 effort=0 velocity=0, mimic joint=left/gripper
- added joint left/i3f: type revolute, parent left/wrist, child left/i3, origin xyz=0.13223 0.0086295 -0.0025 rpy=-1.0408E-15 -5.7778E-30 -5.5511E-15, axis 0 -1 0, limit lower=0 upper=0.8 effort=0 velocity=0, mimic joint=left/gripper
- added joint left/i4f: type revolute, parent left/wrist, child left/i4, origin xyz=0.13046 0.023543 -0.0025 rpy=-1.0408E-15 1.4051E-16 0.13418, axis 0 -1 0, limit lower=0 upper=0.8 effort=0 velocity=0, mimic joint=left/gripper
- added joint left/i5f: type revolute, parent left/wrist, child left/i5, origin xyz=0.12703 0.037692 -0.0025 rpy=1.9429E-14 -3.8109E-15 0.19369, axis 0 -1 0, limit lower=0 upper=0.8 effort=0 velocity=0, mimic joint=left/gripper
- added joint left/shoulder_pitch: type revolute, parent left/shoulder, child left/upperarm_preroll, origin xyz=-0.024 -0.17679 8.6827E-05 rpy=0 0 0, axis -1 0 0, limit lower=-0.15 upper=1.1 effort=0 velocity=0
- added joint left/shoulder_pitch_back_pulley_joint: type fixed, parent left/shoulder_preroll, child left/shoulder_pitch_back_pulley, origin xyz=-0.067526 -0.024095 0.044 rpy=0 0 0, axis 0 0 0
- added joint left/shoulder_pitch_pulley_front_joint: type fixed, parent left/shoulder_preroll, child left/shoulder_pitch_front_pulley, origin xyz=0.067474 -0.024095 0.044 rpy=0 0 0, axis 0 0 0
- added joint left/shoulder_roll: type revolute, parent left/shoulder_preroll, child left/shoulder, origin xyz=-2.6378E-05 0.057605 0.1302 rpy=0 0 0, axis 0 -1 0, limit lower=-0.95 upper=2.3 effort=0 velocity=0
- added joint left/shoulder_roll_bottom_pulley: type fixed, parent left/shoulder, child left/shoulder_roll_bottom_pulley, origin xyz=-0.0208 -0.06848 -0.043 rpy=0 0 0, axis 0 0 -1, limit effort=0 velocity=0
- added joint left/shoulder_roll_top_pulley_joint: type fixed, parent left/shoulder, child left/shoulder_roll_top_pulley, origin xyz=0.0208 -0.06848 0.043 rpy=0 0 0, axis 0 0 0
- added joint left/shoulder_yaw: type revolute, parent left/base_link, child left/shoulder_preroll, origin xyz=-0.00027025 -0.10997 0.008 rpy=0 0 0, axis 0 0 1, limit lower=-0.75 upper=1 effort=0 velocity=0
- added joint left/upperarm_biceps_pulley_joint: type fixed, parent left/upperarm, child left/upperarm_biceps_pulley, origin xyz=0.0375 0 -0.10243 rpy=0 0 0, axis 0 0 0
- added joint left/upperarm_roll: type revolute, parent left/upperarm_preroll, child left/upperarm, origin xyz=0.056992 -0.010088 -0.035587 rpy=0 0 0, axis 0 0 -1, limit lower=-1.56 upper=1.56 effort=0 velocity=0
- added joint left/upperarm_triceps_pulley_joint: type fixed, parent left/upperarm, child left/upperarm_triceps_pulley, origin xyz=-0.0435 0 -0.12843 rpy=0 0 0, axis -1 0 0, limit effort=0 velocity=0
- added joint left/wrist_pitch: type revolute, parent left/lowerarm, child left/wrist, origin xyz=0.1511 -0.01935 0.0048471 rpy=0 0 0, axis 0 1 0, limit lower=-1 upper=1 effort=0 velocity=0
- joint leftbase_displacement: child left_base_link -> left/base_link; origin xyz=-0.2 0 0 rpy=-3.14 0 0 -> xyz=0.2 0 0 rpy=0 0 0

File: xacro/gummi_base.srdf.xacro (robot description, xacro)
@@ -1,50 +1,50 @@
 <?xml version="1.0" ?>
 <robot name="gummi" xmlns:xacro="http://www.ros.org/wiki/xacro">
-  <!-- group name="left_arm" -->
-      <!-- <chain left_base_link="left_base_link" tip_link="left_hand" /> -->
+  <!-- group name="left/arm" -->
+      <!-- <chain left/base_link="left/base_link" tip_link="left/hand" /> -->
 <xacro:macro name="group_left_arm_base">
-  <joint name="left_shoulder_yaw" />
-  <joint name="left_shoulder_roll" />
-  <joint name="left_shoulder_pitch" />
-  <joint name="left_upperarm_roll" />
-  <joint name="left_elbow" />
-  <joint name="left_fastswitch" />
+  <joint name="left/shoulder_yaw" />
+  <joint name="left/shoulder_roll" />
+  <joint name="left/shoulder_pitch" />
+  <joint name="left/upperarm_roll" />
+  <joint name="left/elbow" />
+  <joint name="left/fastswitch" />
 </xacro:macro>
 <xacro:macro name="group_state_left_arm_base">
-  <joint name="left_shoulder_pitch" value="0" />
-  <joint name="left_shoulder_roll" value="0" />
-  <joint name="left_shoulder_yaw" value="0" />
-  <joint name="left_upperarm_roll" value="0" />
-  <joint name="left_elbow" value="0" />
+  <joint name="left/shoulder_pitch" value="0" />
+  <joint name="left/shoulder_roll" value="0" />
+  <joint name="left/shoulder_yaw" value="0" />
+  <joint name="left/upperarm_roll" value="0" />
+  <joint name="left/elbow" value="0" />
 </xacro:macro>
 <xacro:macro name="virtual_joints_base">
   <!--VIRTUAL JOINT: Purpose: this element defines a virtual joint between a robot link and an external frame of reference (considered fixed with respect to the robot)-->
-  <virtual_joint name="virtual_joint" type="fixed" parent_frame="map" child_link="left_base_link" />
+  <virtual_joint name="virtual_joint" type="fixed" parent_frame="map" child_link="left/base_link" />
 </xacro:macro>
 <xacro:macro name="disable_collisions_base">
   <!--DISABLE COLLISIONS: By default it is assumed that any link of the robot could potentially come into collision with any other link in the robot. This tag disables collision checking between a specified pair of links. -->
-  <disable_collisions link1="left_base_link" link2="left_shoulder" reason="Never" />
-  <disable_collisions link1="left_base_link" link2="left_shoulder_preroll" reason="Adjacent" />
-  <disable_collisions link1="left_base_link" link2="left_upperarm" reason="Never" />
-  <disable_collisions link1="left_base_link" link2="left_upperarm_preroll" reason="Never" />
-  <disable_collisions link1="left_shoulder" link2="left_shoulder_preroll" reason="Adjacent" />
-  <disable_collisions link1="left_shoulder" link2="left_upperarm" reason="Never" />
-  <disable_collisions link1="left_shoulder" link2="left_upperarm_preroll" reason="Adjacent" />
-  <disable_collisions link1="left_shoulder_preroll" link2="left_upperarm" reason="Never" />
-  <disable_collisions link1="left_shoulder_preroll" link2="left_upperarm_preroll" reason="Never" />
-  <disable_collisions link1="left_upperarm" link2="left_upperarm_preroll" reason="Adjacent" />
+  <disable_collisions link1="left/base_link" link2="left/shoulder" reason="Never" />
+  <disable_collisions link1="left/base_link" link2="left/shoulder_preroll" reason="Adjacent" />
+  <disable_collisions link1="left/base_link" link2="left/upperarm" reason="Never" />
+  <disable_collisions link1="left/base_link" link2="left/upperarm_preroll" reason="Never" />
+  <disable_collisions link1="left/shoulder" link2="left/shoulder_preroll" reason="Adjacent" />
+  <disable_collisions link1="left/shoulder" link2="left/upperarm" reason="Never" />
+  <disable_collisions link1="left/shoulder" link2="left/upperarm_preroll" reason="Adjacent" />
+  <disable_collisions link1="left/shoulder_preroll" link2="left/upperarm" reason="Never" />
+  <disable_collisions link1="left/shoulder_preroll" link2="left/upperarm_preroll" reason="Never" />
+  <disable_collisions link1="left/upperarm" link2="left/upperarm_preroll" reason="Adjacent" />
 </xacro:macro>
 <xacro:macro name="disable_collisions_mixed">
   <!--MIXED DISABLE COLLISIONS FOR BASE EE COLISIONS: set by hand or remove! -->
-  <disable_collisions link1="left_base_link" link2="left_lowerarm_preroll_u" reason="Never" />
-  <disable_collisions link1="left_lowerarm" link2="left_shoulder" reason="Never" />
-  <disable_collisions link1="left_lowerarm" link2="left_shoulder_preroll" reason="Never" />
-  <disable_collisions link1="left_lowerarm" link2="left_upperarm" reason="Never" />
-  <disable_collisions link1="left_lowerarm" link2="left_upperarm_preroll" reason="Never" />
-  <disable_collisions link1="left_lowerarm_preroll_u" link2="left_shoulder" reason="Never" />
-  <disable_collisions link1="left_lowerarm_preroll_u" link2="left_shoulder_preroll" reason="Never" />
-  <disable_collisions link1="left_lowerarm_preroll_u" link2="left_upperarm" reason="Adjacent" />
-  <disable_collisions link1="left_lowerarm_preroll_u" link2="left_upperarm_preroll" reason="Never" />
-  <disable_collisions link1="left_lowerarm_preroll_u" link2="left_lowerarm_preroll_d" reason="Adjacent" />
+  <disable_collisions link1="left/base_link" link2="left/lowerarm_preroll_u" reason="Never" />
+  <disable_collisions link1="left/lowerarm" link2="left/shoulder" reason="Never" />
+  <disable_collisions link1="left/lowerarm" link2="left/shoulder_preroll" reason="Never" />
+  <disable_collisions link1="left/lowerarm" link2="left/upperarm" reason="Never" />
+  <disable_collisions link1="left/lowerarm" link2="left/upperarm_preroll" reason="Never" />
+  <disable_collisions link1="left/lowerarm_preroll_u" link2="left/shoulder" reason="Never" />
+  <disable_collisions link1="left/lowerarm_preroll_u" link2="left/shoulder_preroll" reason="Never" />
+  <disable_collisions link1="left/lowerarm_preroll_u" link2="left/upperarm" reason="Adjacent" />
+  <disable_collisions link1="left/lowerarm_preroll_u" link2="left/upperarm_preroll" reason="Never" />
+  <disable_collisions link1="left/lowerarm_preroll_u" link2="left/lowerarm_preroll_d" reason="Adjacent" />
 </xacro:macro>
 </robot>

File: xacro/gummi_description.urdf.xacro (robot description, xacro)
@@ -6,7 +6,7 @@
 <link name="base_link"/>
 <joint name="leftbase_displacement" type="fixed">
-  <origin rpy="-3.14 0 0" xyz="-0.2 0 0"/>
+  <origin rpy="0 0 0" xyz="0.2 0 0"/>
   <parent link="base_link"/>
-  <child link="left_base_link"/>
+  <child link="left/base_link"/>
   <axis xyz="0 0 0"/>
 </joint>
