Commit message: changes for namespaceing /left

File: xacro/gummi_description_base.urdf.xacro (robot description, xacro)
@@ -2,5 +2,5 @@
 <robot>
   <link
-    name="left_base_link">
+    name="left/base_link">
     <inertial>
       <origin
@@ -23,5 +23,5 @@
       <geometry>
         <mesh
-          filename="package://gummi_leftbase_$(env ROS_GUMMI_LEFTBASE)/meshes/left_base_link.STL" />
+          filename="package://gummi_leftbase_$(env ROS_GUMMI_LEFTBASE)/meshes/base_link.STL" />
       </geometry>
       <material
@@ -37,10 +37,10 @@
       <geometry>
         <mesh
-          filename="package://gummi_leftbase_$(env ROS_GUMMI_LEFTBASE)/meshes/left_base_link.STL" />
-      </geometry>
-    </collision>
-  </link>
-  <link
-    name="left_shoulder_preroll">
+          filename="package://gummi_leftbase_$(env ROS_GUMMI_LEFTBASE)/meshes/base_link.STL" />
+      </geometry>
+    </collision>
+  </link>
+  <link
+    name="left/shoulder_preroll">
     <inertial>
       <origin
@@ -63,24 +63,24 @@
       <geometry>
         <mesh
-          filename="package://gummi_leftbase_$(env ROS_GUMMI_LEFTBASE)/meshes/left_shoulder_preroll.STL" />
-      </geometry>
-      <material
-        name="">
-        <color
-          rgba="0.79216 0.81961 0.93333 1" />
-      </material>
-    </visual>
-    <collision>
-      <origin
-        xyz="0 0 0"
-        rpy="0 0 0" />
-      <geometry>
-        <mesh
-          filename="package://gummi_leftbase_$(env ROS_GUMMI_LEFTBASE)/meshes/left_shoulder_preroll.STL" />
-      </geometry>
-    </collision>
-  </link>
-  <joint
-    name="left_shoulder_yaw"
+          filename="package://gummi_leftbase_$(env ROS_GUMMI_LEFTBASE)/meshes/shoulder_preroll.STL" />
+      </geometry>
+      <material
+        name="">
+        <color
+          rgba="0.79216 0.81961 0.93333 1" />
+      </material>
+    </visual>
+    <collision>
+      <origin
+        xyz="0 0 0"
+        rpy="0 0 0" />
+      <geometry>
+        <mesh
+          filename="package://gummi_leftbase_$(env ROS_GUMMI_LEFTBASE)/meshes/shoulder_preroll.STL" />
+      </geometry>
+    </collision>
+  </link>
+  <joint
+    name="left/shoulder_yaw"
     type="revolute">
     <origin
@@ -88,7 +88,7 @@
       rpy="0 0 0" />
     <parent
-      link="left_base_link" />
-    <child
-      link="left_shoulder_preroll" />
+      link="left/base_link" />
+    <child
+      link="left/shoulder_preroll" />
     <axis
       xyz="0 0 1" />
@@ -100,5 +100,5 @@
   </joint>
   <link
-    name="left_shoulder">
+    name="left/shoulder">
     <inertial>
       <origin
@@ -121,24 +121,24 @@
       <geometry>
         <mesh
-          filename="package://gummi_leftbase_$(env ROS_GUMMI_LEFTBASE)/meshes/left_shoulder.STL" />
-      </geometry>
-      <material
-        name="">
-        <color
-          rgba="0.79216 0.81961 0.93333 1" />
-      </material>
-    </visual>
-    <collision>
-      <origin
-        xyz="0 0 0"
-        rpy="0 0 0" />
-      <geometry>
-        <mesh
-          filename="package://gummi_leftbase_$(env ROS_GUMMI_LEFTBASE)/meshes/left_shoulder.STL" />
-      </geometry>
-    </collision>
-  </link>
-  <joint
-    name="left_shoulder_roll"
+          filename="package://gummi_leftbase_$(env ROS_GUMMI_LEFTBASE)/meshes/shoulder.STL" />
+      </geometry>
+      <material
+        name="">
+        <color
+          rgba="0.79216 0.81961 0.93333 1" />
+      </material>
+    </visual>
+    <collision>
+      <origin
+        xyz="0 0 0"
+        rpy="0 0 0" />
+      <geometry>
+        <mesh
+          filename="package://gummi_leftbase_$(env ROS_GUMMI_LEFTBASE)/meshes/shoulder.STL" />
+      </geometry>
+    </collision>
+  </link>
+  <joint
+    name="left/shoulder_roll"
     type="revolute">
     <origin
@@ -146,7 +146,7 @@
       rpy="0 0 0" />
     <parent
-      link="left_shoulder_preroll" />
-    <child
-      link="left_shoulder" />
+      link="left/shoulder_preroll" />
+    <child
+      link="left/shoulder" />
     <axis
       xyz="0 -1 0" />
@@ -158,5 +158,5 @@
   </joint>
   <link
-    name="left_upperarm_preroll">
+    name="left/upperarm_preroll">
     <inertial>
       <origin
@@ -179,24 +179,24 @@
       <geometry>
         <mesh
-          filename="package://gummi_leftbase_$(env ROS_GUMMI_LEFTBASE)/meshes/left_upperarm_preroll.STL" />
-      </geometry>
-      <material
-        name="">
-        <color
-          rgba="0.79216 0.81961 0.93333 1" />
-      </material>
-    </visual>
-    <collision>
-      <origin
-        xyz="0 0 0"
-        rpy="0 0 0" />
-      <geometry>
-        <mesh
-          filename="package://gummi_leftbase_$(env ROS_GUMMI_LEFTBASE)/meshes/left_upperarm_preroll.STL" />
-      </geometry>
-    </collision>
-  </link>
-  <joint
-    name="left_shoulder_pitch"
+          filename="package://gummi_leftbase_$(env ROS_GUMMI_LEFTBASE)/meshes/upperarm_preroll.STL" />
+      </geometry>
+      <material
+        name="">
+        <color
+          rgba="0.79216 0.81961 0.93333 1" />
+      </material>
+    </visual>
+    <collision>
+      <origin
+        xyz="0 0 0"
+        rpy="0 0 0" />
+      <geometry>
+        <mesh
+          filename="package://gummi_leftbase_$(env ROS_GUMMI_LEFTBASE)/meshes/upperarm_preroll.STL" />
+      </geometry>
+    </collision>
+  </link>
+  <joint
+    name="left/shoulder_pitch"
     type="revolute">
     <origin
@@ -204,7 +204,7 @@
       rpy="0 0 0" />
     <parent
-      link="left_shoulder" />
-    <child
-      link="left_upperarm_preroll" />
+      link="left/shoulder" />
+    <child
+      link="left/upperarm_preroll" />
     <axis
       xyz="-1 0 0" />
@@ -216,5 +216,5 @@
   </joint>
   <link
-    name="left_upperarm">
+    name="left/upperarm">
     <inertial>
       <origin
@@ -237,24 +237,24 @@
       <geometry>
         <mesh
-          filename="package://gummi_leftbase_$(env ROS_GUMMI_LEFTBASE)/meshes/left_upperarm.STL" />
-      </geometry>
-      <material
-        name="">
-        <color
-          rgba="0.79216 0.81961 0.93333 1" />
-      </material>
-    </visual>
-    <collision>
-      <origin
-        xyz="0 0 0"
-        rpy="0 0 0" />
-      <geometry>
-        <mesh
-          filename="package://gummi_leftbase_$(env ROS_GUMMI_LEFTBASE)/meshes/left_upperarm.STL" />
-      </geometry>
-    </collision>
-  </link>
-  <joint
-    name="left_upperarm_roll"
+          filename="package://gummi_leftbase_$(env ROS_GUMMI_LEFTBASE)/meshes/upperarm.STL" />
+      </geometry>
+      <material
+        name="">
+        <color
+          rgba="0.79216 0.81961 0.93333 1" />
+      </material>
+    </visual>
+    <collision>
+      <origin
+        xyz="0 0 0"
+        rpy="0 0 0" />
+      <geometry>
+        <mesh
+          filename="package://gummi_leftbase_$(env ROS_GUMMI_LEFTBASE)/meshes/upperarm.STL" />
+      </geometry>
+    </collision>
+  </link>
+  <joint
+    name="left/upperarm_roll"
     type="revolute">
     <origin
@@ -262,7 +262,7 @@
       rpy="0 0 0" />
     <parent
-      link="left_upperarm_preroll" />
-    <child
-      link="left_upperarm" />
+      link="left/upperarm_preroll" />
+    <child
+      link="left/upperarm" />
     <axis
       xyz="0 0 -1" />
@@ -274,5 +274,5 @@
   </joint>
   <link
-    name="left_lowerarm_preroll_u">
+    name="left/lowerarm_preroll_u">
     <inertial>
       <origin
@@ -295,24 +295,24 @@
       <geometry>
         <mesh
-          filename="package://gummi_leftbase_$(env ROS_GUMMI_LEFTBASE)/meshes/left_lowerarm_preroll_u.STL" />
-      </geometry>
-      <material
-        name="">
-        <color
-          rgba="0.79216 0.81961 0.93333 1" />
-      </material>
-    </visual>
-    <collision>
-      <origin
-        xyz="0 0 0"
-        rpy="0 0 0" />
-      <geometry>
-        <mesh
-          filename="package://gummi_leftbase_$(env ROS_GUMMI_LEFTBASE)/meshes/left_lowerarm_preroll_u.STL" />
-      </geometry>
-    </collision>
-  </link>
-  <joint
-    name="left_elbow"
+          filename="package://gummi_leftbase_$(env ROS_GUMMI_LEFTBASE)/meshes/lowerarm_preroll_u.STL" />
+      </geometry>
+      <material
+        name="">
+        <color
+          rgba="0.79216 0.81961 0.93333 1" />
+      </material>
+    </visual>
+    <collision>
+      <origin
+        xyz="0 0 0"
+        rpy="0 0 0" />
+      <geometry>
+        <mesh
+          filename="package://gummi_leftbase_$(env ROS_GUMMI_LEFTBASE)/meshes/lowerarm_preroll_u.STL" />
+      </geometry>
+    </collision>
+  </link>
+  <joint
+    name="left/elbow"
     type="revolute">
     <origin
@@ -320,7 +320,7 @@
       rpy="0 0 0" />
     <parent
-      link="left_upperarm" />
-    <child
-      link="left_lowerarm_preroll_u" />
+      link="left/upperarm" />
+    <child
+      link="left/lowerarm_preroll_u" />
     <axis
       xyz="0 -1 0" />
@@ -332,5 +332,5 @@
   </joint>
   <link
-    name="left_upperarm_biceps_pulley">
+    name="left/upperarm_biceps_pulley">
     <inertial>
       <origin
@@ -353,24 +353,24 @@
       <geometry>
         <mesh
-          filename="package://gummi_leftbase_$(env ROS_GUMMI_LEFTBASE)/meshes/left_upperarm_biceps_pulley.STL" />
-      </geometry>
-      <material
-        name="">
-        <color
-          rgba="0.79216 0.81961 0.93333 1" />
-      </material>
-    </visual>
-    <collision>
-      <origin
-        xyz="0 0 0"
-        rpy="0 0 0" />
-      <geometry>
-        <mesh
-          filename="package://gummi_leftbase_$(env ROS_GUMMI_LEFTBASE)/meshes/left_upperarm_biceps_pulley.STL" />
-      </geometry>
-    </collision>
-  </link>
-  <joint
-    name="left_upperarm_biceps_pulley_joint"
+          filename="package://gummi_leftbase_$(env ROS_GUMMI_LEFTBASE)/meshes/upperarm_biceps_pulley.STL" />
+      </geometry>
+      <material
+        name="">
+        <color
+          rgba="0.79216 0.81961 0.93333 1" />
+      </material>
+    </visual>
+    <collision>
+      <origin
+        xyz="0 0 0"
+        rpy="0 0 0" />
+      <geometry>
+        <mesh
+          filename="package://gummi_leftbase_$(env ROS_GUMMI_LEFTBASE)/meshes/upperarm_biceps_pulley.STL" />
+      </geometry>
+    </collision>
+  </link>
+  <joint
+    name="left/upperarm_biceps_pulley_joint"
     type="fixed">
     <origin
@@ -378,12 +378,12 @@
       rpy="0 0 0" />
     <parent
-      link="left_upperarm" />
-    <child
-      link="left_upperarm_biceps_pulley" />
+      link="left/upperarm" />
+    <child
+      link="left/upperarm_biceps_pulley" />
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